File: KiCad/Device/Device.kicad_pcb (KiCad board)
At the start: 2 copper layers, 0 parts

Commit message: Opdatering af switches
Parts:
- added C1: 1uF, Capacitor_THT:C_Disc_D5.0mm_W2.5mm_P5.00mm, F.Cu at (170.2, 91.4)
- added C2: 20pF, Capacitor_THT:C_Disc_D5.0mm_W2.5mm_P5.00mm, F.Cu at (119.9, 114.7)
- added C3: 20pF, Capacitor_THT:C_Disc_D5.0mm_W2.5mm_P5.00mm, F.Cu at (170.2, 87.4)
- added C4: 200n, Capacitor_THT:C_Disc_D5.0mm_W2.5mm_P5.00mm, F.Cu at (148.0, 112.6)
- added D1: RødLED, LED_THT:LED_D3.0mm_FlatTop, F.Cu at (178.4, 87.4)
- added D2: GrønLED, LED_THT:LED_D3.0mm_FlatTop, F.Cu at (186.3, 78.8)
- added D3: BZX79C3V3, Diode_SMD:D_MELF_Handsoldering, F.Cu at (167.6, 81.3)
- added IC1: ATTINY167-XUR, Package_DIP:DIP-20_W7.62mm_Socket, F.Cu at (179.1, 92.7)
- added J1: Mikrofon, Connector_Phoenix_MC_HighVoltage:PhoenixContact_MCV_1,5_2-G-5.08_1x02_P5.08mm_Vertical, F.Cu at (109.2, 88.9)
- added J2: Lysføler, Connector_PinSocket_2.54mm:PinSocket_2x01_P2.54mm_Vertical, F.Cu at (111.8, 76.2)
- added J3: Optisk sensor, Connector_PinSocket_2.54mm:PinSocket_2x02_P2.54mm_Vertical, F.Cu at (111.8, 99.1)
- added J4: Fugtføler, Connector_PinSocket_2.54mm:PinSocket_1x03_P2.54mm_Vertical, F.Cu at (106.7, 109.2)
- added J5: VCC, Connector_Phoenix_MC_HighVoltage:PhoenixContact_MCV_1,5_2-G-5.08_1x02_P5.08mm_Vertical, F.Cu at (149.9, 73.7)
- added J6: ESP8266(wifi), Connector_PinSocket_2.54mm:PinSocket_2x04_P2.54mm_Vertical, F.Cu at (196.9, 95.3)
- added R1: 10k, Resistor_THT:R_Axial_DIN0309_L9.0mm_D3.2mm_P12.70mm_Horizontal, F.Cu at (147.5, 83.2)
- added R2: 2.2k, Resistor_THT:R_Axial_DIN0309_L9.0mm_D3.2mm_P12.70mm_Horizontal, F.Cu at (135.8, 87.9)
- added R3: 10k, Resistor_THT:R_Axial_DIN0309_L9.0mm_D3.2mm_P12.70mm_Horizontal, F.Cu at (131.7, 97.4)
- added R4: 100k, Resistor_THT:R_Axial_DIN0309_L9.0mm_D3.2mm_P12.70mm_Horizontal, F.Cu at (147.5, 78.4)
- added R5: 1k, Resistor_THT:R_Axial_DIN0309_L9.0mm_D3.2mm_P12.70mm_Horizontal, F.Cu at (131.7, 78.4)
- added R6: 1k, Resistor_THT:R_Axial_DIN0309_L9.0mm_D3.2mm_P12.70mm_Horizontal, F.Cu at (119.9, 105.5)
- added R7: 200, Resistor_THT:R_Axial_DIN0309_L9.0mm_D3.2mm_P12.70mm_Horizontal, F.Cu at (131.7, 83.2)
- added R8: 200, Resistor_THT:R_Axial_DIN0309_L9.0mm_D3.2mm_P12.70mm_Horizontal, F.Cu at (119.9, 110.3)
- added R9: 15, Resistor_THT:R_Axial_DIN0309_L9.0mm_D3.2mm_P12.70mm_Horizontal, F.Cu at (131.7, 92.7)
- added SW1: SW_MEC_5E, Button_Switch_THT:SW_PUSH_6mm_H4.3mm, F.Cu at (161.8, 107.0)
- added SW3: SW_MEC_5E, Button_Switch_THT:SW_PUSH_6mm_H4.3mm, F.Cu at (149.2, 104.1)
- added SW4: SW_DIP_x02, Button_Switch_THT:SW_DIP_SPSTx02_Slide_9.78x7.26mm_W7.62mm_P2.54mm, F.Cu at (120.7, 80.0)
- added Y1: Crystal, Crystal:Crystal_HC18-U_Vertical, F.Cu at (193.0, 111.8)
