File: KiCad/Device/Device.kicad_sch (KiCad schematic)
At the start: 4 parts, among them IC1 ATTINY167-XUR, J1 Conn_02x04_Odd_Even

Commit message: device tilføjelse
Parts:
- removed J? (x2): Conn_01x10_MountingPin, Connector_PinHeader_2.54mm:PinHeader_1x10_P2.54mm_Vertical, symbol Connector_Generic_MountingPin:Conn_01x10_MountingPin
- added C?: (no value), symbol Device:C
- added J1, J?: Screw_Terminal_01x02, symbol Connector:Screw_Terminal_01x02
- added R?: (no value), symbol Device:R
- renumbered J1 to J2
Connections:
- net GPIO2 is gone; now on net SCL: J2.3 (Pin_3)
- net SPI_CS2 is gone; now on net SDA: J2.5 (Pin_5)
- net GND: now also IC1.6 (AGND), J1.1 (Pin_1), J?.1 (Pin_1)
- net Mic_out: now reaches IC1.1 (PA0/RXLIN/RXD/ADC0/PCINT0)
- net Mic_out: now also C?.2
- net VCC: now reaches IC1.5 (AVCC)
- net VCC: now also J?.2 (Pin_2), R?.2
- net SDA: now reaches IC1.20 (PB0/SDA/DI/OCR1AU/PCINT8)
- net SCL: now reaches IC1.18 (PB2/SCL/USCK/OC1AV/PCINT10)
- net PD&EN renamed EN
- net RXD: no longer names the net of J2.7 (Pin_7)
- net TXD: no longer names the net of J2.2 (Pin_2)
- new net: C?.1, J1.2 (Pin_2), R?.1
- no-connect marks 0 -> 2
Other:
- moved on the sheet: J2

Commit message: Device tilføjelser
Parts:
- added C2, C3: (no value), symbol Device:C
- added D1, D?: (no value), symbol Device:LED
- added J2: (no value), symbol Connector_Generic:Conn_02x01
- added J3: (no value), symbol Connector_Generic:Conn_02x02_Odd_Even
- added J4: (no value), symbol Connector_Generic:Conn_01x03
- added R1: 10k, symbol Device:R
- added R3, R4, R? (x2): (no value), symbol Device:R
- added R?: 1k, symbol Device:R
- added SW?: (no value), symbol Switch:SW_DIP_x01
- added SW?: (no value), Button_Switch_SMD:SW_MEC_5GSH9, symbol Switch:SW_MEC_5G
- added SW?: (no value), symbol Switch:SW_MEC_5G
- added Y1: (no value), symbol Device:Crystal
- C1: renamed from C?; value (none) -> 1uF
- J1: value Screw_Terminal_01x02 -> (none)
- J5: renamed from J?; value Screw_Terminal_01x02 -> (none)
- J6: renamed from J2; value Conn_02x04_Odd_Even -> (none)
- R2: renamed from R?; value (none) -> 2.2k
Connections:
- net GND: now also IC1.16 (GND), C2.2, C3.2, D1.1 (K), J4.1 (Pin_1), R1.2, R3.2, R4.2, R?.2, SW?.1 (A), SW?.2 (A)
- net Mic_out: now also IC1.3 (PA2/MISO/DO/OC0A/ADC2/PCINT2); no longer IC1.1 (PA0/RXLIN/RXD/ADC0/PCINT0)
- net Reset: now also IC1.11 (PB7/DW/~{RESET}/OC1BX/ADC10/PCINT15), R?.1, SW?.3 (B), SW?.4 (B)
- net VCC: no longer IC1.5 (AVCC), J5.2 (Pin_2)
- net GrønLED: now reaches IC1.12 (PB6/INT0/OC1AX/ADC9/PCINT14)
- net GrønLED: now also R?.2
- net XTAL2: now reaches IC1.13 (PB5/CLKO/XTAL2/OC1BW/ADC8/PCINT13)
- net XTAL2: now also C3.1, Y1.2
- net XTAL1: now reaches IC1.14 (PB4/CLKI/XTAL1/OC1AW/PCINT12)
- net XTAL1: now also C2.1, Y1.1
- net +5V: now reaches IC1.15 (VCC)
- net +5V: now also IC1.5 (AVCC), D1.2 (A), D?.2 (A), J2.2 (Pin_2), J3.1 (Pin_1), J3.2 (Pin_2), J4.3 (Pin_3), R?.2, SW?.1 (A), SW?.2, SW?.2 (A)
- net Button01: now reaches IC1.19 (PB1/DO/OC1BU/PCINT9)
- net Button01: now also R?.1, SW?.3 (B), SW?.4 (B)
- net Photo_out: now reaches IC1.4 (PA3/INT1/ISRC/ADC3/PCINT3)
- net Photo_out: now also J2.1 (Pin_1), R1.1
- net Fugt_out: now reaches IC1.7 (PA4/MOSI/SDA/DI/ICP1/ADC4/PCINT4)
- net Fugt_out: now also J4.2 (Pin_2)
- net Op.Sensor_out: now reaches IC1.8 (PA5/SCK/SCL/USCK/T1/ADC5/PCINT5)
- net Op.Sensor_out: now also J3.4 (Pin_4), R4.1
- new net: J5.2 (Pin_2), SW?.1
- new net: D?.1 (K), R?.1
- new net: J3.3 (Pin_3), R3.1
- no-connect marks 2 -> 7
Other:
- note added: "Knapper"
- note added: "Occilator - 16MHz"
- note added: "Sensorer"
- moved on the sheet: C1, IC1, J1, J5, J6, R2

Commit message: Update Device.kicad_sch
Parts:
- C2, C3: value (none) -> 20pF
- D1: value (none) -> RødLED
- D?: value (none) -> GrønLED
- J1: value (none) -> Mikrofon
- J2: value (none) -> Lysføler
- J3: value (none) -> Optisk sensor
- J4: value (none) -> Fugtføler
- J5: value (none) -> VCC
- J6: value (none) -> ESP8266(wifi)
- R3: value (none) -> 10k
- R4: value (none) -> 100k
- R?: value (none) -> 1k
- R?: value (none) -> R
- SW?: value (none) -> SW_DIP_x01
- SW?: value (none) -> Button01
- SW?: value (none) -> Reset; footprint (none) -> Button_Switch_SMD:SW_MEC_5GSH9
- Y1: value (none) -> Crystal
Other:
- note added: "LED'er"
- moved on the sheet: D1, D?, J5, J6, R?, SW?

Commit message: kicad device fodlister
Parts:
- gave numbers to parts that had none: 7
Changed lines of the file:
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@@
   (symbol (lib_id "Switch:SW_DIP_x01") (at 160.02 30.48 0) (unit 1)
     (in_bom yes) (on_board yes) (fields_autoplaced)
-    (property "Reference" "SW?" (id 0) (at 160.02 22.86 0))
+    (property "Reference" "SW3" (id 0) (at 160.02 22.86 0))
     (property "Value" "SW_DIP_x01" (id 1) (at 160.02 25.4 0))
     (property "Footprint" "" (id 2) (at 160.02 30.48 0)
@@
   (symbol (lib_id "Device:LED") (at 204.47 97.79 180) (unit 1)
     (in_bom yes) (on_board yes)
-    (property "Reference" "D?" (id 0) (at 198.755 92.075 0)
+    (property "Reference" "D2" (id 0) (at 198.755 92.075 0)
       (effects (font (size 1.27 1.27)) (justify right))
     )
@@
   (symbol (lib_id "power:GND") (at 105.41 99.06 270) (unit 1)
     (in_bom yes) (on_board yes) (fields_autoplaced)
-    (property "Reference" "#PWR?" (id 0) (at 99.06 99.06 0)
+    (property "Reference" "#PWR0123" (id 0) (at 99.06 99.06 0)
       (effects (font (size 1.27 1.27)) hide)
     )
@@
   (symbol (lib_id "Device:R") (at 158.75 102.87 0) (unit 1)
     (in_bom yes) (on_board yes) (fields_autoplaced)
-    (property "Reference" "R?" (id 0) (at 161.29 101.5999 0)
+    (property "Reference" "R6" (id 0) (at 161.29 101.5999 0)
       (effects (font (size 1.27 1.27)) (justify left))
     )
@@
   (symbol (lib_id "power:GND") (at 158.75 106.68 0) (unit 1)
     (in_bom yes) (on_board yes)
-    (property "Reference" "#PWR?" (id 0) (at 158.75 113.03 0)
+    (property "Reference" "#PWR0121" (id 0) (at 158.75 113.03 0)
       (effects (font (size 1.27 1.27)) hide)
     )
@@
   (symbol (lib_id "Device:R") (at 118.11 104.14 0) (unit 1)
     (in_bom yes) (on_board yes) (fields_autoplaced)
-    (property "Reference" "R?" (id 0) (at 120.65 102.8699 0)
+    (property "Reference" "R5" (id 0) (at 120.65 102.8699 0)
       (effects (font (size 1.27 1.27)) (justify left))
     )
@@
   (symbol (lib_id "power:+5V") (at 118.11 107.95 180) (unit 1)
     (in_bom yes) (on_board yes)
-    (property "Reference" "#PWR?" (id 0) (at 118.11 104.14 0)
+    (property "Reference" "#PWR0122" (id 0) (at 118.11 104.14 0)
       (effects (font (size 1.27 1.27)) hide)
     )
@@
   (symbol (lib_id "Device:R") (at 214.63 97.79 90) (unit 1)
     (in_bom yes) (on_board yes) (fields_autoplaced)
-    (property "Reference" "R?" (id 0) (at 214.63 91.44 90))
+    (property "Reference" "R7" (id 0) (at 214.63 91.44 90))
     (property "Value" "R" (id 1) (at 214.63 93.98 90))
     (property "Footprint" "" (id 2) (at 214.63 99.568 90)
@@
   (symbol (lib_id "Switch:SW_MEC_5G") (at 149.86 99.06 0) (unit 1)
     (in_bom yes) (on_board yes) (fields_autoplaced)
-    (property "Reference" "SW?" (id 0) (at 149.86 91.44 0))
+    (property "Reference" "SW2" (id 0) (at 149.86 91.44 0))
     (property "Value" "Button01" (id 1) (at 149.86 93.98 0))
     (property "Footprint" "Button_Switch_SMD:SW_MEC_5GSH9" (id 2) (at 149.86 93.98 0)
@@
   (symbol (lib_id "Switch:SW_MEC_5G") (at 110.49 99.06 0) (unit 1)
     (in_bom yes) (on_board yes) (fields_autoplaced)
-    (property "Reference" "SW?" (id 0) (at 110.49 91.44 0))
+    (property "Reference" "SW1" (id 0) (at 110.49 91.44 0))
     (property "Value" "Reset" (id 1) (at 110.49 93.98 0))
     (property "Footprint" "Button_Switch_SMD:SW_MEC_5GSH9" (id 2) (at 110.49 93.98 0)
@@
   (symbol (lib_id "power:+5V") (at 144.78 99.06 90) (unit 1)
     (in_bom yes) (on_board yes)
-    (property "Reference" "#PWR?" (id 0) (at 148.59 99.06 0)
+    (property "Reference" "#PWR0124" (id 0) (at 148.59 99.06 0)
       (effects (font (size 1.27 1.27)) hide)
     )
@@
   (symbol (lib_id "power:+5V") (at 201.93 97.79 90) (unit 1)
     (in_bom yes) (on_board yes)
-    (property "Reference" "#PWR?" (id 0) (at 205.74 97.79 0)
+    (property "Reference" "#PWR0120" (id 0) (at 205.74 97.79 0)
       (effects (font (size 1.27 1.27)) hide)
     )
@@
       (reference "#PWR0119") (unit 1) (value "+5V") (footprint "")
     )
+    (path "/fea08acc-7035-4e5b-a922-5743506308d1"
+      (reference "#PWR0120") (unit 1) (value "+5V") (footprint "")
+    )
+    (path "/4a27a9f5-4020-4f2a-a146-7d6090273db9"
+      (reference "#PWR0121") (unit 1) (value "GND") (footprint "")
+    )
+    (path "/7a30d29d-a709-4147-90ef-8a1f600bf705"
+      (reference "#PWR0122") (unit 1) (value "+5V") (footprint "")
+    )
     (path "/2f18d0ed-287a-40e1-8d53-20e0b4160484"
-      (reference "#PWR?") (unit 1) (value "GND") (footprint "")
-    )
-    (path "/4a27a9f5-4020-4f2a-a146-7d6090273db9"
-      (reference "#PWR?") (unit 1) (value "GND") (footprint "")
-    )
-    (path "/7a30d29d-a709-4147-90ef-8a1f600bf705"
-      (reference "#PWR?") (unit 1) (value "+5V") (footprint "")
+      (reference "#PWR0123") (unit 1) (value "GND") (footprint "")
     )
     (path "/f572accc-c719-48ce-a6b9-1254ff3d0e9d"
-      (reference "#PWR?") (unit 1) (value "+5V") (footprint "")
-    )
-    (path "/fea08acc-7035-4e5b-a922-5743506308d1"
-      (reference "#PWR?") (unit 1) (value "+5V") (footprint "")
+      (reference "#PWR0124") (unit 1) (value "+5V") (footprint "")
     )
     (path "/c3859b88-ee1c-4daa-9fe4-63386a16086c"
-      (reference "C1") (unit 1) (value "1uF") (footprint "")
+      (reference "C1") (unit 1) (value "1uF") (footprint "Capacitor_THT:C_Disc_D5.0mm_W2.5mm_P5.00mm")
     )
     (path "/649d19fd-cb36-4c8b-b96a-635864303db2"
-      (reference "C2") (unit 1) (value "20pF") (footprint "")
+      (reference "C2") (unit 1) (value "20pF") (footprint "Capacitor_THT:C_Disc_D5.0mm_W2.5mm_P5.00mm")
     )
     (path "/7d94699e-7c95-4848-8c16-b3aa311edd29"
-      (reference "C3") (unit 1) (value "20pF") (footprint "")
+      (reference "C3") (unit 1) (value "20pF") (footprint "Capacitor_THT:C_Disc_D5.0mm_W2.5mm_P5.00mm")
     )
     (path "/7611e2c8-7c51-45ab-a61a-212ad250d6ba"
-      (reference "D1") (unit 1) (value "RødLED") (footprint "")
+      (reference "D1") (unit 1) (value "RødLED") (footprint "LED_THT:LED_D3.0mm_FlatTop")
     )
     (path "/2543488b-3564-4a07-8bac-d5d9882c70ff"
-      (reference "D?") (unit 1) (value "GrønLED") (footprint "")
+      (reference "D2") (unit 1) (value "GrønLED") (footprint "LED_THT:LED_D3.0mm_FlatTop")
     )
     (path "/ed8a7f02-cf05-41d0-97b4-4388ef205e73"
@@
     )
     (path "/a340ffec-ed73-4437-8fbf-7434d84e9c5c"
-      (reference "J1") (unit 1) (value "Mikrofon") (footprint "")
+      (reference "J1") (unit 1) (value "Mikrofon") (footprint "Connector_Phoenix_MC_HighVoltage:PhoenixContact_MCV_1,5_2-G-5.08_1x02_P5.08mm_Vertical")
     )
     (path "/077e27cc-b774-4fc3-be0f-1a8a82f9f441"
@@
     )
     (path "/9dde5f18-d33a-482b-aed4-9f855bdb6d54"
-      (reference "J5") (unit 1) (value "VCC") (footprint "")
+      (reference "J5") (unit 1) (value "VCC") (footprint "Connector_Phoenix_MC_HighVoltage:PhoenixContact_MCV_1,5_2-G-5.08_1x02_P5.08mm_Vertical")
     )
     (path "/f959907b-1cef-4760-b043-4260a660a2ae"
@@
     )
     (path "/de92152a-3f95-470e-8a68-519c1291418b"
-      (reference "R1") (unit 1) (value "10k") (footprint "")
+      (reference "R1") (unit 1) (value "10k") (footprint "Resistor_THT:R_Axial_DIN0309_L9.0mm_D3.2mm_P12.70mm_Horizontal")
     )
     (path "/d8200a86-aa75-47a3-ad2a-7f4c9c999a6f"
-      (reference "R2") (unit 1) (value "2.2k") (footprint "")
+      (reference "R2") (unit 1) (value "2.2k") (footprint "Resistor_THT:R_Axial_DIN0309_L9.0mm_D3.2mm_P12.70mm_Horizontal")
     )
     (path "/fd863afb-816b-4205-b430-34a1463e0b1e"
-      (reference "R3") (unit 1) (value "10k") (footprint "")
+      (reference "R3") (unit 1) (value "10k") (footprint "Resistor_THT:R_Axial_DIN0309_L9.0mm_D3.2mm_P12.70mm_Horizontal")
     )
     (path "/83b62012-b8ad-4a46-8b52-85c03aeb73ba"
-      (reference "R4") (unit 1) (value "100k") (footprint "")
+      (reference "R4") (unit 1) (value "100k") (footprint "Resistor_THT:R_Axial_DIN0309_L9.0mm_D3.2mm_P12.70mm_Horizontal")
+    )
+    (path "/57e99af3-a41a-446e-b28a-0272c5c10ec2"
+      (reference "R5") (unit 1) (value "1k") (footprint "Resistor_THT:R_Axial_DIN0309_L9.0mm_D3.2mm_P12.70mm_Horizontal")
     )
     (path "/330e4a4e-1686-411b-941a-e77769eb093d"
-      (reference "R?") (unit 1) (value "1k") (footprint "")
-    )
-    (path "/57e99af3-a41a-446e-b28a-0272c5c10ec2"
-      (reference "R?") (unit 1) (value "1k") (footprint "")
+      (reference "R6") (unit 1) (value "1k") (footprint "Resistor_THT:R_Axial_DIN0309_L9.0mm_D3.2mm_P12.70mm_Horizontal")
     )
     (path "/a2014450-1b0f-4962-a973-f42e00681deb"
-      (reference "R?") (unit 1) (value "R") (footprint "")
+      (reference "R7") (unit 1) (value "R") (footprint "Resistor_THT:R_Axial_DIN0309_L9.0mm_D3.2mm_P12.70mm_Horizontal")
+    )
+    (path "/cd4f78c6-1905-45bc-8353-13fa5b012b26"
+      (reference "SW1") (unit 1) (value "Reset") (footprint "Button_Switch_SMD:SW_MEC_5GSH9")
+    )
+    (path "/bb081121-b10a-47df-8559-7a1d3f99d968"
+      (reference "SW2") (unit 1) (value "Button01") (footprint "Button_Switch_SMD:SW_MEC_5GSH9")
     )
     (path "/1f9cef0e-84ac-4eda-84fc-9f00d1d3d7b1"
-      (reference "SW?") (unit 1) (value "SW_DIP_x01") (footprint "")
-    )
-    (path "/bb081121-b10a-47df-8559-7a1d3f99d968"
-      (reference "SW?") (unit 1) (value "Button01") (footprint "Button_Switch_SMD:SW_MEC_5GSH9")
-    )
-    (path "/cd4f78c6-1905-45bc-8353-13fa5b012b26"
-      (reference "SW?") (unit 1) (value "Reset") (footprint "Button_Switch_SMD:SW_MEC_5GSH9")
+      (reference "SW3") (unit 1) (value "SW_DIP_x01") (footprint "")
     )
     (path "/5df0654c-8d6d-486d-b5f4-0be0de8af6ef"
