File: KiCad/Device/Device.kicad_sch (KiCad schematic)
At the start: 30 parts, among them IC1 ATTINY167-XUR, J1 Mikrofon, J2 Lysføler, J3 Optisk sensor, J4 Fugtføler, J5 VCC, J6 ESP8266(wifi), J7 Conn_02x06_Odd_Even, SW1 SW_MEC_5E, SW3 SW_MEC_5E, SW4 SW_DIP_x02, Y1 Crystal

Commit message: Update Device.kicad_sch
Parts:
- R1: value (none) -> 2k
Changed lines of the file:
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@@
       (effects (font (size 1.27 1.27)) (justify left))
     )
-    (property "Value" "" (id 1) (at 99.06 64.7699 0)
+    (property "Value" "2k" (id 1) (at 99.06 64.7699 0)
       (effects (font (size 1.27 1.27)) (justify left))
     )

Commit message: Opdateret connecter 5v
Parts:
- J7: footprint Connector_PinHeader_2.54mm:PinHeader_2x06_P2.54mm_Vertical -> (none)
Changed lines of the file:
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@@
     (property "Reference" "J7" (id 0) (at 250.19 111.76 0))
     (property "Value" "Conn_02x06_Odd_Even" (id 1) (at 250.19 114.3 0))
-    (property "Footprint" "Connector_PinHeader_2.54mm:PinHeader_2x06_P2.54mm_Vertical" (id 2) (at 248.92 123.19 0)
+    (property "Footprint" "" (id 2) (at 248.92 123.19 0)
       (effects (font (size 1.27 1.27)) hide)
     )
@@
     )
     (path "/bcb4dcbe-acea-49b0-8634-f95f0474cdf9"
-      (reference "J7") (unit 1) (value "Conn_02x06_Odd_Even") (footprint "Connector_PinHeader_2.54mm:PinHeader_2x06_P2.54mm_Vertical")
+      (reference "J7") (unit 1) (value "Conn_02x06_Odd_Even") (footprint "Connector_PinHeader_2.54mm:PinHeader_2x06_P2.54mm_Horizontal")
     )
     (path "/de92152a-3f95-470e-8a68-519c1291418b"

Commit message: kicad
Parts:
- C4: value 200n -> (none)
- J7: footprint (none) -> Connector_PinHeader_2.54mm:PinHeader_2x06_P2.54mm_Horizontal
Connections:
- net UP7 is gone; now on net MIC: C1.2, IC1.11 (PA7/AREF/XREF/AIN1ADC7/PCINT7), J7.10 (Pin_10)
- net +3V3: no longer D3.1 (K)
- net +5V: now also D3.1 (K)
- net MIC: no longer C1.1, J1.2 (Pin_2), R2.1
- new net: C1.1, J1.2 (Pin_2), R2.1
Other:
- moved on the sheet: D3, R10

Commit message: Update Device.kicad_sch
Parts:
- C4: value (none) -> 100pF
Other:
- note added: "Spændingsregulator"
- note removed: "Strømforsyning"
- moved on the sheet: J6, R11, R12
