File: KiCad/HUB/HUB.kicad_sch (KiCad schematic)
At the start: 2 parts, among them J1 ESP8266(wifi)

Commit message: hub
Parts:
- added D?: GrønLED, LED_THT:LED_D3.0mm_FlatTop, symbol Device:LED
- added R1: 200, Resistor_THT:R_Axial_DIN0309_L9.0mm_D3.2mm_P12.70mm_Horizontal, symbol Device:R
- added R? (x2): 1k, Resistor_THT:R_Axial_DIN0309_L9.0mm_D3.2mm_P12.70mm_Horizontal, symbol Device:R
- added SW1, SW2: SW_MEC_5E, Button_Switch_THT:SW_PUSH_6mm_H4.3mm, symbol Switch:SW_MEC_5E
Connections:
- net +3V3: now also IC1.40 (VBUS)
- net GND: now also R1.2, R?.2, R?.2
- net Button01: now reaches IC1.3 (PA00)
- net Button01: now also R?.1, SW1.2 (K)
- net Data+: now reaches IC1.38 (DP)
- net Data-: now reaches IC1.39 (DM)
- net Button02: now reaches IC1.4 (PA01)
- net Button02: now also R?.1, SW2.2 (K)
- net LED_G: now reaches IC1.5 (PA02)
- net LED_G: now also D?.2 (A)
- net USB renamed USB_VBOF
- net USB1 renamed USB_ID
- new net: D?.1 (K), R1.1
- new net +5V: SW1.1 (2), SW2.1 (2)
Other:
- note added: "Knapper"
- note added: "LED"

Commit message: HUB_Schematic_done
Parts:
- added J2: (no value), symbol Connector:USB_B_Mini
- added R?: 1k, Resistor_THT:R_Axial_DIN0309_L9.0mm_D3.2mm_P12.70mm_Horizontal, symbol Device:R
- added SW?: SW_MEC_5E, Button_Switch_THT:SW_PUSH_6mm_H4.3mm, symbol Switch:SW_MEC_5E
- IC1: value (none) -> AT32UC3B164-AUT; footprint (none) -> QFP50P900X900X120-48N
- R1: value 200 -> (none)
- gave numbers to parts that had none: 1
Connections:
- net +5V is gone; now on net +3V3: SW1.1 (2), SW2.1 (2)
- net +3V3: now also IC1.15 (VDDANA), IC1.17 (VDDIN), IC1.24 (VDDIO_1), IC1.36 (VDDIO_2), IC1.48 (VDDIO_3), J2.1 (VBUS), R?.2
- net Data+: now also J2.3 (D+)
- net Data-: now also J2.2 (D-)
- net GND: now also IC1.13 (GNDANA), IC1.19 (GND_2), IC1.37 (GND_3), J2.5 (GND), J2.6 (Shield), SW?.1 (2)
- net Reset: now also IC1.47 (RESET_N), R?.1, SW?.2 (K)
- net USB_ID: now also J2.4 (ID)
- net at IC1.16 (VDDOUT): now also IC1.18 (VDDCORE_2), IC1.41 (VDDPLL), IC1.42 (VDDCORE_3), IC1.6 (VDDCORE_1)

Commit message: Næsten_færdigt_pcb
Parts:
- IC1: footprint QFP50P900X900X120-48N -> (none)
- J2: value (none) -> USB_B_Mini
- R1: value (none) -> 150
- gave numbers to parts that had none: 4
Connections:
- net at IC1.16 (VDDOUT), IC1.41 (VDDPLL), IC1.42 (VDDCORE_3)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: no longer IC1.18 (VDDCORE_2)

Commit message: hub
Parts:
- IC1: footprint (none) -> user:QFP50P900X900X120-48N
- J2: footprint (none) -> Connector_USB:USB_Mini-B_Lumberg_2486_01_Horizontal
Other:
- moved on the sheet: J1, J2
